Commit message: fix inertias and lengths to be 7l

File: fanuc_lrmate200id_support/urdf/lrmate200id7l.transmission.xacro (robot description, xacro)
@@ -34,8 +34,7 @@
     <type>transmission_interface/SimpleTransmission</type>
     <joint name="joint_1">
-      <hardwareInterface>PositionJointInterface</hardwareInterface>
+              <hardwareInterface>hardware_interface/PositionJointInterface</hardwareInterface>
     </joint>
     <actuator name="motor_1">
-      <hardwareInterface>PositionJointInterface</hardwareInterface>
       <mechanicalReduction>1</mechanicalReduction>
     </actuator>
@@ -44,8 +43,7 @@
     <type>transmission_interface/SimpleTransmission</type>
     <joint name="joint_2">
-      <hardwareInterface>PositionJointInterface</hardwareInterface>
+              <hardwareInterface>hardware_interface/PositionJointInterface</hardwareInterface>
     </joint>
     <actuator name="motor_2">
-      <hardwareInterface>PositionJointInterface</hardwareInterface>
       <mechanicalReduction>1</mechanicalReduction>
     </actuator>
@@ -54,8 +52,7 @@
     <type>transmission_interface/SimpleTransmission</type>
     <joint name="joint_3">
-      <hardwareInterface>PositionJointInterface</hardwareInterface>
+              <hardwareInterface>hardware_interface/PositionJointInterface</hardwareInterface>
     </joint>
     <actuator name="motor_3">
-      <hardwareInterface>PositionJointInterface</hardwareInterface>
       <mechanicalReduction>1</mechanicalReduction>
     </actuator>
@@ -64,8 +61,7 @@
     <type>transmission_interface/SimpleTransmission</type>
     <joint name="joint_4">
-      <hardwareInterface>PositionJointInterface</hardwareInterface>
+              <hardwareInterface>hardware_interface/PositionJointInterface</hardwareInterface>
     </joint>
     <actuator name="motor_4">
-      <hardwareInterface>PositionJointInterface</hardwareInterface>
       <mechanicalReduction>1</mechanicalReduction>
     </actuator>
@@ -74,8 +70,7 @@
     <type>transmission_interface/SimpleTransmission</type>
     <joint name="joint_5">
-      <hardwareInterface>PositionJointInterface</hardwareInterface>
+              <hardwareInterface>hardware_interface/PositionJointInterface</hardwareInterface>
     </joint>
     <actuator name="motor_5">
-      <hardwareInterface>PositionJointInterface</hardwareInterface>
       <mechanicalReduction>1</mechanicalReduction>
     </actuator>
@@ -84,8 +79,7 @@
     <type>transmission_interface/SimpleTransmission</type>
     <joint name="joint_6">
-      <hardwareInterface>PositionJointInterface</hardwareInterface>
+              <hardwareInterface>hardware_interface/PositionJointInterface</hardwareInterface>
     </joint>
     <actuator name="motor_6">
-      <hardwareInterface>PositionJointInterface</hardwareInterface>
       <mechanicalReduction>1</mechanicalReduction>
     </actuator>

File: fanuc_lrmate200id_support/urdf/lrmate200id7l_macro.xacro (robot description, xacro)
@@ -2,245 +2,213 @@
 <robot xmlns:xacro="http://ros.org/wiki/xacro">
   <xacro:include filename="$(find fanuc_resources)/urdf/common_materials.xacro"/>
-<!--  <xacro:include filename="$(find fanuc_resources)/urdf/common_constants.xacro"/>-->
   <xacro:include filename="$(find fanuc_lrmate200id_support)/urdf/lrmate200id7l.transmission.xacro" />
-  <!-- Inertia parameters -->
-  <property name="base_link_mass" value="6.215" />  <!-- This mass might be incorrect -->
-  <property name="link_1_mass" value="2.13" />
-  <property name="link_2_mass" value="7.65" />
-  <property name="link_3_mass" value="2.91" />
-  <property name="link_4_mass" value="3.70" />
-  <property name="link_5_mass" value="1.70" />
-  <property name="link_6_mass" value="0.137" />  <!-- This mass might be incorrect -->
-  <xacro:macro name="fanuc_lrmate200id7l" params="prefix">
-    <link name="${prefix}base_link">
-      <visual>
-        <origin xyz="0 0 0" rpy="0 0 0"/>
-        <geometry>
-          <mesh filename="package://fanuc_lrmate200id_support/meshes/lrmate200id/visual/base_link.stl"/>
-        </geometry>
-        <xacro:material_fanuc_gray28 />
-      </visual>
-      <collision>
-        <origin xyz="0 0 0" rpy="0 0 0"/>
-        <geometry>
-          <mesh filename="package://fanuc_lrmate200id_support/meshes/lrmate200id/collision/base_link.stl"/>
-        </geometry>
-      </collision>
-      <inertial>
-        <origin xyz="0 0 0" rpy="0 0 0"/>
-        <mass value="${base_link_mass}"/>
-        <!-- Copied from abb_irb120t https://github.com/ros-industrial/abb_experimental/blob/indigo-devel/abb_irb120_support/urdf/irb120t_macro.xacro. -->
-        <inertia ixx="0.0247272" ixy="-8.0784E-05" ixz="0.00130902" iyy="0.0491285" iyz="-8.0419E-06" izz="0.0472376"/>
-      </inertial>
-    </link>
-    <link name="${prefix}link_1">
-      <visual>
-        <origin xyz="0 0 0" rpy="0 0 0"/>
-        <geometry>
-          <mesh filename="package://fanuc_lrmate200id_support/meshes/lrmate200id/visual/link_1.stl"/>
-        </geometry>
-        <xacro:material_fanuc_yellow />
-      </visual>
-      <collision>
-        <origin xyz="0 0 0" rpy="0 0 0"/>
-        <geometry>
-          <mesh filename="package://fanuc_lrmate200id_support/meshes/lrmate200id/collision/link_1.stl"/>
-        </geometry>
-      </collision>
-      <inertial>
-        <origin xyz="-0.000010 -0.054550 0.028725" rpy="0 0 0"/>
-        <mass value="${link_1_mass}"/>
-        <!-- Estimated with Meshlab and stl model. '600' is the scale to make inertial to be standard values
-             refering abb_irb120t https://github.com/ros-industrial/abb_experimental/blob/indigo-devel/abb_irb120_support/urdf/irb120t_macro.xacro. -->
-        <inertia
-          ixx="${600 * 0.000048}" ixy="0.0" ixz="${600 * -0.000006}"
-          iyy="${600 * 0.000035}" iyz="0.0" izz="${600 * 0.000037}"/>
-      </inertial>
-    </link>
-    <link name="${prefix}link_2">
-      <visual>
-        <origin xyz="0 0 0" rpy="0 0 0"/>
-        <geometry>
-          <mesh filename="package://fanuc_lrmate200id_support/meshes/lrmate200id/visual/link_2.stl"/>
-        </geometry>
-        <xacro:material_fanuc_yellow />
-      </visual>
-      <collision>
-        <origin xyz="0 0 0" rpy="0 0 0"/>
-        <geometry>
-          <mesh filename="package://fanuc_lrmate200id_support/meshes/lrmate200id/collision/link_2.stl"/>
-        </geometry>
-      </collision>
-      <inertial>
-        <origin xyz="-0.002701 -0.000977 0.159466" rpy="0 0 0"/>
-        <mass value="${link_2_mass}"/>
-        <inertia
-          ixx="${600 * 0.000182}" ixy="0.0" ixz="0.0"
-          iyy="${600 * 0.000157}" iyz="${600 * -0.000001}"
-          izz="${600 * 0.000049}"/>
-      </inertial>
-    </link>
-    <link name="${prefix}link_3">
-      <visual>
-        <origin xyz="0 0 0" rpy="0 0 0"/>
-        <geometry>
-          <mesh filename="package://fanuc_lrmate200id_support/meshes/lrmate200id/visual/link_3.stl"/>
-        </geometry>
-        <xacro:material_fanuc_yellow />
-      </visual>
-      <collision>
-        <origin xyz="0 0 0" rpy="0 0 0"/>
-        <geometry>
-          <mesh filename="package://fanuc_lrmate200id_support/meshes/lrmate200id/collision/link_3.stl"/>
-        </geometry>
-      </collision>
-      <inertial>
-        <origin xyz="-0.000065 0.017074 0.008866" rpy="0 0 0"/>
-        <mass value="${link_3_mass}"/>
-        <inertia
-          ixx="${600 * 0.000007}" ixy="0.0" ixz="${600 * -0.000001}"
-          iyy="${600 * 0.000008}" iyz="0.0"
-          izz="${600 * 0.000008}"/>
-      </inertial>
-    </link>
-    <link name="${prefix}link_4">
-      <visual>
-        <origin xyz="0 0 0" rpy="0 0 0"/>
-        <geometry>
-          <mesh filename="package://fanuc_lrmate200id_support/meshes/lrmate200id/visual/link_4.stl"/>
-        </geometry>
-        <xacro:material_fanuc_yellow />
-      </visual>
-      <collision>
-        <origin xyz="0 0 0" rpy="0 0 0"/>
-        <geometry>
-          <mesh filename="package://fanuc_lrmate200id_support/meshes/lrmate200id/collision/link_4.stl"/>
-        </geometry>
-      </collision>
-      <inertial>
-        <origin xyz="0.000067 0.002203 0.221634" rpy="0 0 0"/>
-        <mass value="${link_4_mass}"/>
-        <inertia
-          ixx="${600 * 0.000005}" ixy="0.0" ixz="0.0"
-          iyy="${600 * 0.000019}" iyz="0.0"
-          izz="${600 * 0.000019}"/>
-      </inertial>
-    </link>
-    <link name="${prefix}link_5">
-      <visual>
-        <origin xyz="0 0 0" rpy="0 0 0"/>
-        <geometry>
-          <mesh filename="package://fanuc_lrmate200id_support/meshes/lrmate200id/visual/link_5.stl"/>
-        </geometry>
-        <xacro:material_fanuc_yellow />
-      </visual>
-      <collision>
-        <origin xyz="0 0 0" rpy="0 0 0"/>
-        <geometry>
-          <mesh filename="package://fanuc_lrmate200id_support/meshes/lrmate200id/collision/link_5.stl"/>
-        </geometry>
-      </collision>
-      <inertial>
-        <origin xyz="-0.000010 -0.054550 0.028725" rpy="0 0 0"/>
-        <mass value="${link_5_mass}"/>
-        <!-- This mass might be incorrect because of nan value of
-             'link_5.stl' in Meshlab inertia estimation. -->
-        <inertia
-          ixx="${600 * 0.00004}" ixy="0.0" ixz="${600 * -0.000004}"
-          iyy="${600 * 0.00003}" iyz="0.0" izz="${600 * 0.00003}"/>
-      </inertial>
-    </link>
-    <link name="${prefix}link_6">
-      <visual>
-        <origin xyz="0 0 0" rpy="0 0 0"/>
-        <geometry>
-          <mesh filename="package://fanuc_lrmate200id_support/meshes/lrmate200id/visual/link_6.stl"/>
-        </geometry>
-        <xacro:material_fanuc_black />
-      </visual>
-      <collision>
-        <origin xyz="0 0 0" rpy="0 0 0"/>
-        <geometry>
-          <mesh filename="package://fanuc_lrmate200id_support/meshes/lrmate200id/collision/link_6.stl"/>
-        </geometry>
-      </collision>
-      <inertial>
-        <origin xyz="-0.000000 0.000000 -0.003006" rpy="0 0 0" />
-        <mass value="${link_6_mass}"/>
-        <inertia
-          ixx="0.01" ixy="0.0" ixz="0.0"
-          iyy="0.01" iyz="0.0"
-          izz="0.01"/>
-      </inertial>
-    </link>
-    <joint name="${prefix}joint_1" type="revolute">
-      <origin xyz="0 0 0.330" rpy="0 0 0" />
-      <parent link="${prefix}base_link" />
-      <child link="${prefix}link_1" />
-      <axis xyz="0 0 1" />
-      <limit effort="0" lower="-2.965" upper="2.965" velocity="7.85" />
-      <dynamics damping="1.0" friction="1.0"/>
-    </joint>
-    <joint name="${prefix}joint_2" type="revolute">
-      <origin xyz="0.050 0 0" rpy="0 0 0"/>
-      <parent link="${prefix}link_1" />
-      <child link="${prefix}link_2" />
-      <axis xyz="0 1 0" />
-      <limit effort="0" lower="-1.745329" upper="2.530727" velocity="6.63" />
-      <dynamics damping="1.0" friction="1.0"/>
-    </joint>
-    <joint name="${prefix}joint_3" type="revolute">
-      <origin xyz="0 0 0.330" rpy="0 0 0"/>
-      <parent link="${prefix}link_2" />
-      <child link="${prefix}link_3" />
-      <axis xyz="0 -1 0" />
-      <limit effort="0" lower="-2.450966" upper="4.886922" velocity="9.08" />
-      <dynamics damping="1.0" friction="1.0"/>
-    </joint>
-    <joint name="${prefix}joint_4" type="revolute">
-      <origin xyz="0 0 0.035" rpy="0 0 0"/>
-      <parent link="${prefix}link_3"/>
-      <child link="${prefix}link_4"/>
-      <axis xyz="-1 0 0"/>
-      <limit effort="0" lower="-3.315" upper="3.315" velocity="9.60" />
-      <dynamics damping="1.0" friction="1.0"/>
-    </joint>
-    <joint name="${prefix}joint_5" type="revolute">
-      <origin xyz="0.335 0 0" rpy="0 0 0"/>
-      <parent link="${prefix}link_4"/>
-      <child link="${prefix}link_5"/>
-      <axis xyz="0 -1 0"/>
-      <limit effort="0" lower="-2.18" upper="2.18" velocity="9.51" />
-      <dynamics damping="1.0" friction="1.0"/>
-    </joint>
-    <joint name="${prefix}joint_6" type="revolute">
-      <origin xyz="0.080 0 0" rpy="0 0 0"/>
-      <parent link="${prefix}link_5"/>
-      <child link="${prefix}link_6"/>
-      <axis xyz="-1 0 0"/>
-      <limit effort="0" lower="-6.285" upper="6.285" velocity="17.45" />
-      <dynamics damping="1.0" friction="1.0"/>
-    </joint>
-    <!-- ROS base_link to Fanuc World Coordinates transform -->
-    <link name="${prefix}base" />
-    <joint name="${prefix}base_link-base" type="fixed">
-      <origin xyz="0 0 0.330" rpy="0 0 0"/>
-      <parent link="${prefix}base_link"/>
-      <child link="${prefix}base"/>
-    </joint>
-    <!-- ROS-Industrial 'flange' frame: attachment point for EEF models -->
-    <link name="${prefix}flange" />
-    <joint name="${prefix}link_6-flange" type="fixed">
-      <origin xyz="0 0 0" rpy="0 0 0" />
-      <parent link="${prefix}link_6" />
-      <child link="${prefix}flange" />
-    </joint>
-    <!-- ROS-Industrial 'tool0' frame: all-zeros tool frame -->
-    <link name="${prefix}tool0" />
-    <joint name="${prefix}flange-tool0" type="fixed">
-      <origin xyz="0 0 0" rpy="${pi} ${-pi/2.0} 0" />
-      <parent link="${prefix}flange" />
-      <child link="${prefix}tool0" />
-    </joint>
-  </xacro:macro>
-</robot>
+  <xacro:macro name="cylinder_inertial" params="radius length mass *origin">
+        <inertial>
+            <mass value="${mass}" />
+            <xacro:insert_block name="origin" />
+            <inertia ixx="${0.0833333 * mass * (3 * radius * radius + length * length)}" ixy="0.0" ixz="0.0"
+            iyy="${0.0833333 * mass * (3 * radius * radius + length * length)}" iyz="0.0"
+            izz="${0.5 * mass * radius * radius}" />
+        </inertial>
+    </xacro:macro>
+    <xacro:macro name="fanuc_lrmate200id7l" params="prefix">
+    <xacro:property name="base_mass" value="4.0" />
+    <xacro:property name="shoulder_mass" value="3.7000" />
+    <xacro:property name="upper_arm_mass" value="8.3930" />
+    <xacro:property name="forearm_mass" value="2.2750" />
+    <xacro:property name="wrist_1_mass" value="1.2190" />
+    <xacro:property name="wrist_2_mass" value="1.2190" />
+    <xacro:property name="wrist_3_mass" value="0.1879" />
+      <!-- links: main serial chain -->
+      <link name="${prefix}base_link">
+        <visual>
+          <origin xyz="0 0 0" rpy="0 0 0"/>
+          <geometry>
+            <mesh filename="package://fanuc_lrmate200id_support/meshes/lrmate200id/visual/base_link.stl"/>
+          </geometry>
+          <xacro:material_fanuc_gray28 />
+        </visual>
+        <collision>
+          <origin xyz="0 0 0" rpy="0 0 0"/>
+          <geometry>
+            <mesh filename="package://fanuc_lrmate200id_support/meshes/lrmate200id/collision/base_link.stl"/>
+          </geometry>
+        </collision>
+        <xacro:cylinder_inertial radius="0.06" length="0.05" mass="${base_mass}">
+            <origin xyz="0.0 0.0 0.0" rpy="0 0 0" />
+        </xacro:cylinder_inertial>
+      </link>
+      <link name="${prefix}link_1">
+        <visual>
+          <origin xyz="0 0 0" rpy="0 0 0"/>
+          <geometry>
+            <mesh filename="package://fanuc_lrmate200id_support/meshes/lrmate200id/visual/link_1.stl"/>
+          </geometry>
+          <xacro:material_fanuc_yellow />
+        </visual>
+        <collision>
+          <origin xyz="0 0 0" rpy="0 0 0"/>
+          <geometry>
+            <mesh filename="package://fanuc_lrmate200id_support/meshes/lrmate200id/collision/link_1.stl"/>
+          </geometry>
+        </collision>
+        <xacro:cylinder_inertial radius="0.06" length="0.15" mass="${shoulder_mass}">
+            <origin xyz="0.0 0.0 0.0" rpy="0 0 0" />
+        </xacro:cylinder_inertial>
+      </link>
+      <link name="${prefix}link_2">
+        <visual>
+          <origin xyz="0 0 0" rpy="0 0 0"/>
+          <geometry>
+            <mesh filename="package://fanuc_lrmate200id_support/meshes/lrmate200id7l/visual/link_2.stl"/>
+          </geometry>
+          <xacro:material_fanuc_yellow />
+        </visual>
+        <collision>
+          <origin xyz="0 0 0" rpy="0 0 0"/>
+          <geometry>
+            <mesh filename="package://fanuc_lrmate200id_support/meshes/lrmate200id7l/collision/link_2.stl"/>
+          </geometry>
+        </collision>
+        <xacro:cylinder_inertial radius="0.06" length="0.56" mass="${upper_arm_mass}">
+            <origin xyz="0.0 0.0 0.28" rpy="0 0 0" />
+        </xacro:cylinder_inertial>
+      </link>
+      <link name="${prefix}link_3">
+        <visual>
+          <origin xyz="0 0 0" rpy="0 0 0"/>
+          <geometry>
+            <mesh filename="package://fanuc_lrmate200id_support/meshes/lrmate200id/visual/link_3.stl"/>
+          </geometry>
+          <xacro:material_fanuc_yellow />
+        </visual>
+        <collision>
+          <origin xyz="0 0 0" rpy="0 0 0"/>
+          <geometry>
+            <mesh filename="package://fanuc_lrmate200id_support/meshes/lrmate200id/collision/link_3.stl"/>
+          </geometry>
+        </collision>
+        <xacro:cylinder_inertial radius="0.06" length="0.5" mass="${forearm_mass}">
+            <origin xyz="0.0 0.0 0.25" rpy="0 0 0" />
+        </xacro:cylinder_inertial>
+      </link>
+      <link name="${prefix}link_4">
+        <visual>
+          <origin xyz="0 0 0" rpy="0 0 0"/>
+          <geometry>
+            <mesh filename="package://fanuc_lrmate200id_support/meshes/lrmate200id7l/visual/link_4.stl"/>
+          </geometry>
+          <xacro:material_fanuc_yellow />
+        </visual>
+        <collision>
+          <origin xyz="0 0 0" rpy="0 0 0"/>
+          <geometry>
+            <mesh filename="package://fanuc_lrmate200id_support/meshes/lrmate200id7l/collision/link_4.stl"/>
+          </geometry>
+        </collision>
+        <xacro:cylinder_inertial radius="0.6" length="0.12" mass="${wrist_1_mass}">
+            <origin xyz="0.0 0.0 0.0" rpy="0 0 0" />
+        </xacro:cylinder_inertial>
+      </link>
+      <link name="${prefix}link_5">
+        <visual>
+          <origin xyz="0 0 0" rpy="0 0 0"/>
+          <geometry>
+            <mesh filename="package://fanuc_lrmate200id_support/meshes/lrmate200id/visual/link_5.stl"/>
+          </geometry>
+          <xacro:material_fanuc_yellow />
+        </visual>
+        <collision>
+          <origin xyz="0 0 0" rpy="0 0 0"/>
+          <geometry>
+            <mesh filename="package://fanuc_lrmate200id_support/meshes/lrmate200id/collision/link_5.stl"/>
+          </geometry>
+        </collision>
+        <xacro:cylinder_inertial radius="0.6" length="0.12" mass="${wrist_2_mass}">
+            <origin xyz="0.0 0.0 0.0" rpy="0 0 0" />
+        </xacro:cylinder_inertial>
+      </link>
+      <link name="${prefix}link_6">
+        <visual>
+          <origin xyz="0 0 0" rpy="0 0 0"/>
+          <geometry>
+            <mesh filename="package://fanuc_lrmate200id_support/meshes/lrmate200id/visual/link_6.stl"/>
+          </geometry>
+          <xacro:material_fanuc_black />
+        </visual>
+        <collision>
+          <origin xyz="0 0 0" rpy="0 0 0"/>
+          <geometry>
+            <mesh filename="package://fanuc_lrmate200id_support/meshes/lrmate200id/collision/link_6.stl"/>
+          </geometry>
+        </collision>
+        <xacro:cylinder_inertial radius="0.6" length="0.12" mass="${wrist_3_mass}">
+            <origin xyz="0.0 0.0 0.0" rpy="0 0 0" />
+        </xacro:cylinder_inertial>
+      </link>
+      <!-- joints: main serial chain -->
+      <joint name="${prefix}joint_1" type="revolute">
+        <origin xyz="0 0 0.330" rpy="0 0 0" />
+        <parent link="${prefix}base_link" />
+        <child link="${prefix}link_1" />
+        <axis xyz="0 0 1" />
+        <limit effort="100" lower="${radians(-170)}" upper="${radians(170)}" velocity="${radians(370)}" />
+      </joint>
+      <joint name="${prefix}joint_2" type="revolute">
+        <origin xyz="0.050 0 0" rpy="0 0 0"/>
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