Commit message: first draft gazebo for 200id

File: fanuc_lrmate200id_support/urdf/lrmate200id7l_macro.xacro (robot description, xacro)
@@ -2,6 +2,15 @@
 <robot xmlns:xacro="http://ros.org/wiki/xacro">
   <xacro:include filename="$(find fanuc_resources)/urdf/common_materials.xacro"/>
+<!--  <xacro:include filename="$(find fanuc_resources)/urdf/common_constants.xacro"/>-->
+  <xacro:include filename="$(find fanuc_lrmate200id_support)/urdf/lrmate200id7l.transmission.xacro" />
+  <!-- Inertia parameters -->
+  <property name="base_link_mass" value="6.215" />  <!-- This mass might be incorrect -->
+  <property name="link_1_mass" value="2.13" />
+  <property name="link_2_mass" value="7.65" />
+  <property name="link_3_mass" value="2.91" />
+  <property name="link_4_mass" value="3.70" />
+  <property name="link_5_mass" value="1.70" />
+  <property name="link_6_mass" value="0.137" />  <!-- This mass might be incorrect -->
   <xacro:macro name="fanuc_lrmate200id7l" params="prefix">
-    <!-- links: main serial chain -->
     <link name="${prefix}base_link">
       <visual>
@@ -18,4 +27,10 @@
         </geometry>
       </collision>
+      <inertial>
+        <origin xyz="0 0 0" rpy="0 0 0"/>
+        <mass value="${base_link_mass}"/>
+        <!-- Copied from abb_irb120t https://github.com/ros-industrial/abb_experimental/blob/indigo-devel/abb_irb120_support/urdf/irb120t_macro.xacro. -->
+        <inertia ixx="0.0247272" ixy="-8.0784E-05" ixz="0.00130902" iyy="0.0491285" iyz="-8.0419E-06" izz="0.0472376"/>
+      </inertial>
     </link>
     <link name="${prefix}link_1">
@@ -33,4 +48,13 @@
         </geometry>
       </collision>
+      <inertial>
+        <origin xyz="-0.000010 -0.054550 0.028725" rpy="0 0 0"/>
+        <mass value="${link_1_mass}"/>
+        <!-- Estimated with Meshlab and stl model. '600' is the scale to make inertial to be standard values
+             refering abb_irb120t https://github.com/ros-industrial/abb_experimental/blob/indigo-devel/abb_irb120_support/urdf/irb120t_macro.xacro. -->
+        <inertia
+          ixx="${600 * 0.000048}" ixy="0.0" ixz="${600 * -0.000006}"
+          iyy="${600 * 0.000035}" iyz="0.0" izz="${600 * 0.000037}"/>
+      </inertial>
     </link>
     <link name="${prefix}link_2">
@@ -38,14 +62,22 @@
         <origin xyz="0 0 0" rpy="0 0 0"/>
         <geometry>
-          <mesh filename="package://fanuc_lrmate200id_support/meshes/lrmate200id7l/visual/link_2.stl"/>
-        </geometry>
-        <xacro:material_fanuc_yellow />
-      </visual>
-      <collision>
-        <origin xyz="0 0 0" rpy="0 0 0"/>
-        <geometry>
-          <mesh filename="package://fanuc_lrmate200id_support/meshes/lrmate200id7l/collision/link_2.stl"/>
-        </geometry>
-      </collision>
+          <mesh filename="package://fanuc_lrmate200id_support/meshes/lrmate200id/visual/link_2.stl"/>
+        </geometry>
+        <xacro:material_fanuc_yellow />
+      </visual>
+      <collision>
+        <origin xyz="0 0 0" rpy="0 0 0"/>
+        <geometry>
+          <mesh filename="package://fanuc_lrmate200id_support/meshes/lrmate200id/collision/link_2.stl"/>
+        </geometry>
+      </collision>
+      <inertial>
+        <origin xyz="-0.002701 -0.000977 0.159466" rpy="0 0 0"/>
+        <mass value="${link_2_mass}"/>
+        <inertia
+          ixx="${600 * 0.000182}" ixy="0.0" ixz="0.0"
+          iyy="${600 * 0.000157}" iyz="${600 * -0.000001}"
+          izz="${600 * 0.000049}"/>
+      </inertial>
     </link>
     <link name="${prefix}link_3">
@@ -63,4 +95,12 @@
         </geometry>
       </collision>
+      <inertial>
+        <origin xyz="-0.000065 0.017074 0.008866" rpy="0 0 0"/>
+        <mass value="${link_3_mass}"/>
+        <inertia
+          ixx="${600 * 0.000007}" ixy="0.0" ixz="${600 * -0.000001}"
+          iyy="${600 * 0.000008}" iyz="0.0"
+          izz="${600 * 0.000008}"/>
+      </inertial>
     </link>
     <link name="${prefix}link_4">
@@ -68,14 +108,22 @@
         <origin xyz="0 0 0" rpy="0 0 0"/>
         <geometry>
-          <mesh filename="package://fanuc_lrmate200id_support/meshes/lrmate200id7l/visual/link_4.stl"/>
-        </geometry>
-        <xacro:material_fanuc_yellow />
-      </visual>
-      <collision>
-        <origin xyz="0 0 0" rpy="0 0 0"/>
-        <geometry>
-          <mesh filename="package://fanuc_lrmate200id_support/meshes/lrmate200id7l/collision/link_4.stl"/>
-        </geometry>
-      </collision>
+          <mesh filename="package://fanuc_lrmate200id_support/meshes/lrmate200id/visual/link_4.stl"/>
+        </geometry>
+        <xacro:material_fanuc_yellow />
+      </visual>
+      <collision>
+        <origin xyz="0 0 0" rpy="0 0 0"/>
+        <geometry>
+          <mesh filename="package://fanuc_lrmate200id_support/meshes/lrmate200id/collision/link_4.stl"/>
+        </geometry>
+      </collision>
+      <inertial>
+        <origin xyz="0.000067 0.002203 0.221634" rpy="0 0 0"/>
+        <mass value="${link_4_mass}"/>
+        <inertia
+          ixx="${600 * 0.000005}" ixy="0.0" ixz="0.0"
+          iyy="${600 * 0.000019}" iyz="0.0"
+          izz="${600 * 0.000019}"/>
+      </inertial>
     </link>
     <link name="${prefix}link_5">
@@ -93,4 +141,13 @@
         </geometry>
       </collision>
+      <inertial>
+        <origin xyz="-0.000010 -0.054550 0.028725" rpy="0 0 0"/>
+        <mass value="${link_5_mass}"/>
+        <!-- This mass might be incorrect because of nan value of
+             'link_5.stl' in Meshlab inertia estimation. -->
+        <inertia
+          ixx="${600 * 0.00004}" ixy="0.0" ixz="${600 * -0.000004}"
+          iyy="${600 * 0.00003}" iyz="0.0" izz="${600 * 0.00003}"/>
+      </inertial>
     </link>
     <link name="${prefix}link_6">
@@ -108,6 +165,13 @@
         </geometry>
       </collision>
-    </link>
-    <!-- joints: main serial chain -->
+      <inertial>
+        <origin xyz="-0.000000 0.000000 -0.003006" rpy="0 0 0" />
+        <mass value="${link_6_mass}"/>
+        <inertia
+          ixx="0.01" ixy="0.0" ixz="0.0"
+          iyy="0.01" iyz="0.0"
+          izz="0.01"/>
+      </inertial>
+    </link>
     <joint name="${prefix}joint_1" type="revolute">
       <origin xyz="0 0 0.330" rpy="0 0 0" />
@@ -115,5 +179,6 @@
       <child link="${prefix}link_1" />
       <axis xyz="0 0 1" />
-      <limit effort="0" lower="${radians(-170)}" upper="${radians(170)}" velocity="${radians(370)}" />
+      <limit effort="0" lower="-2.965" upper="2.965" velocity="7.85" />
+      <dynamics damping="1.0" friction="1.0"/>
     </joint>
     <joint name="${prefix}joint_2" type="revolute">
@@ -122,12 +187,14 @@
       <child link="${prefix}link_2" />
       <axis xyz="0 1 0" />
-      <limit effort="0" lower="${radians(-100)}" upper="${radians(145)}" velocity="${radians(310)}" />
+      <limit effort="0" lower="-1.745329" upper="2.530727" velocity="6.63" />
+      <dynamics damping="1.0" friction="1.0"/>
     </joint>
     <joint name="${prefix}joint_3" type="revolute">
-      <origin xyz="0 0 0.440" rpy="0 0 0"/>
+      <origin xyz="0 0 0.330" rpy="0 0 0"/>
       <parent link="${prefix}link_2" />
       <child link="${prefix}link_3" />
       <axis xyz="0 -1 0" />
-      <limit effort="0" lower="${radians(-70)}" upper="${radians(213)}" velocity="${radians(410)}" />
+      <limit effort="0" lower="-2.450966" upper="4.886922" velocity="9.08" />
+      <dynamics damping="1.0" friction="1.0"/>
     </joint>
     <joint name="${prefix}joint_4" type="revolute">
@@ -136,12 +203,14 @@
       <child link="${prefix}link_4"/>
       <axis xyz="-1 0 0"/>
-      <limit effort="0" lower="${radians(-190)}" upper="${radians(190)}" velocity="${radians(550)}" />
+      <limit effort="0" lower="-3.315" upper="3.315" velocity="9.60" />
+      <dynamics damping="1.0" friction="1.0"/>
     </joint>
     <joint name="${prefix}joint_5" type="revolute">
-      <origin xyz="0.420 0 0" rpy="0 0 0"/>
+      <origin xyz="0.335 0 0" rpy="0 0 0"/>
       <parent link="${prefix}link_4"/>
       <child link="${prefix}link_5"/>
       <axis xyz="0 -1 0"/>
-      <limit effort="0" lower="${radians(-125)}" upper="${radians(125)}" velocity="${radians(545)}" />
+      <limit effort="0" lower="-2.18" upper="2.18" velocity="9.51" />
+      <dynamics damping="1.0" friction="1.0"/>
     </joint>
     <joint name="${prefix}joint_6" type="revolute">
@@ -150,7 +219,8 @@
       <child link="${prefix}link_6"/>
       <axis xyz="-1 0 0"/>
-      <limit effort="0" lower="${radians(-360)}" upper="${radians(360)}" velocity="${radians(1000)}" />
-    </joint>
-    <!-- ROS-Industrial 'base' frame: base_link to Fanuc World Coordinates transform -->
+      <limit effort="0" lower="-6.285" upper="6.285" velocity="17.45" />
+      <dynamics damping="1.0" friction="1.0"/>
+    </joint>
+    <!-- ROS base_link to Fanuc World Coordinates transform -->
     <link name="${prefix}base" />
     <joint name="${prefix}base_link-base" type="fixed">

Commit message: copy velocities from mh5

File: fanuc_lrmate200id_support/urdf/lrmate200id7l_macro.xacro (robot description, xacro)
@@ -153,5 +153,5 @@
         <child link="${prefix}link_1" />
         <axis xyz="0 0 1" />
-        <limit effort="100" lower="${radians(-170)}" upper="${radians(170)}" velocity="${radians(370)}" />
+        <limit effort="100" lower="${radians(-170)}" upper="${radians(170)}" velocity="2.96" />
       </joint>
       <joint name="${prefix}joint_2" type="revolute">
@@ -160,5 +160,5 @@
         <child link="${prefix}link_2" />
         <axis xyz="0 1 0" />
-        <limit effort="100" lower="${radians(-100)}" upper="${radians(145)}" velocity="${radians(310)}" />
+        <limit effort="100" lower="${radians(-100)}" upper="${radians(145)}" velocity="2.96" />
       </joint>
       <joint name="${prefix}joint_3" type="revolute">
@@ -167,5 +167,5 @@
         <child link="${prefix}link_3" />
         <axis xyz="0 -1 0" />
-        <limit effort="100" lower="${radians(-70)}" upper="${radians(213)}" velocity="${radians(410)}" />
+        <limit effort="100" lower="${radians(-70)}" upper="${radians(213)}" velocity="2.96" />
       </joint>
       <joint name="${prefix}joint_4" type="revolute">
@@ -174,5 +174,5 @@
         <child link="${prefix}link_4"/>
         <axis xyz="-1 0 0"/>
-        <limit effort="100" lower="${radians(-190)}" upper="${radians(190)}" velocity="${radians(550)}" />
+        <limit effort="100" lower="${radians(-190)}" upper="${radians(190)}" velocity="3.48" />
       </joint>
       <joint name="${prefix}joint_5" type="revolute">
@@ -181,5 +181,5 @@
         <child link="${prefix}link_5"/>
         <axis xyz="0 -1 0"/>
-        <limit effort="100" lower="${radians(-125)}" upper="${radians(125)}" velocity="${radians(545)}" />
+        <limit effort="100" lower="${radians(-125)}" upper="${radians(125)}" velocity="3.48" />
       </joint>
       <joint name="${prefix}joint_6" type="revolute">
@@ -188,5 +188,5 @@
         <child link="${prefix}link_6"/>
         <axis xyz="-1 0 0"/>
-        <limit effort="100" lower="${radians(-360)}" upper="${radians(360)}" velocity="${radians(1000)}" />
+        <limit effort="100" lower="${radians(-360)}" upper="${radians(360)}" velocity="6.97" />
       </joint>
       <!-- ROS-Industrial 'base' frame: base_link to Fanuc World Coordinates transform -->
